Commit message: added nav2 params and launch, fixed robor urdf

File: src/rover_bringup/urdf/rover.urdf (robot description, URDF)
Before this commit: robot rover_bot, 3 links, 2 joints
Links:
- removed link laser_frame
- added link left_wheel; visual cylinder length=0.07 radius=0.096
- added link right_wheel; visual cylinder length=0.07 radius=0.096
- link base_link: geometry visual box size=0.5 0.4 0.17
Joints:
- removed joint laser_joint
- added joint left_wheel_joint: type fixed, parent base_link, child left_wheel, origin xyz=0.15 0.235 -0.035 rpy=0 0 0, axis 0 1 0
- added joint right_wheel_joint: type fixed, parent base_link, child right_wheel, origin xyz=0.15 -0.235 -0.035 rpy=0 0 0, axis 0 1 0

Commit message: ADD imu_link and 4x4 to rover.urdf

File: src/rover_bringup/urdf/rover.urdf (robot description, URDF)
Before this commit: robot rover_bot, 4 links, 3 joints
Links:
- removed link left_wheel
- removed link right_wheel
- added link front_left_wheel; visual cylinder length=0.07 radius=0.096
- added link front_right_wheel; visual cylinder length=0.07 radius=0.096
- added link gps_link; visual box size=0.05 0.05 0.02
- added link imu_link; visual box size=0.05 0.05 0.02
- added link rear_left_wheel; visual cylinder length=0.07 radius=0.096
- added link rear_right_wheel; visual cylinder length=0.07 radius=0.096
Joints:
- removed joint left_wheel_joint
- removed joint right_wheel_joint
- added joint front_left_wheel_joint: type fixed, parent base_link, child front_left_wheel, origin xyz=0.15 0.235 -0.035 rpy=0 0 0, axis 0 1 0
- added joint front_right_wheel_joint: type fixed, parent base_link, child front_right_wheel, origin xyz=0.15 -0.235 -0.035 rpy=0 0 0, axis 0 1 0
- added joint gps_joint: type fixed, parent base_link, child gps_link, origin xyz=0.39 0 0.1 rpy=0 0 0
- added joint imu_joint: type fixed, parent base_link, child imu_link, origin xyz=0.15 0 0.1 rpy=0 0 0
- added joint rear_left_wheel_joint: type fixed, parent base_link, child rear_left_wheel, origin xyz=-0.15 0.235 -0.035 rpy=0 0 0, axis 0 1 0
- added joint rear_right_wheel_joint: type fixed, parent base_link, child rear_right_wheel, origin xyz=-0.15 -0.235 -0.035 rpy=0 0 0, axis 0 1 0
